File: Templates/Template Project/Template Project.kicad_pcb (KiCad board)
At the start: 4 copper layers, 0 parts

Commit message: Migration to KiCad 6
Other:
- net class Default removed
Changed lines of the file:
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@@
-(kicad_pcb (version 20171130) (host pcbnew "(5.1.6)-1")
+(kicad_pcb (version 20211014) (generator pcbnew)
   (general
     (thickness 1.6)
-    (drawings 0)
-    (tracks 0)
-    (zones 0)
-    (modules 0)
-    (nets 1)
   )
-  (page A4)
+  (paper "A4")
   (title_block
     (title "<PCB Name>")
     (date "<Issue Date>")
-    (rev <Revision>)
+    (rev "<Revision>")
     (company "<Not Used>")
     (comment 1 "<Drawn By>")
@@
   )
   (layers
-    (0 Top.Copper signal)
-    (1 Plane.1 power)
-    (2 Plane.2 power)
-    (31 Bottom.Copper signal)
-    (34 B.Paste user)
-    (35 F.Paste user)
-    (36 B.SilkS user)
-    (37 F.SilkS user)
-    (38 B.Mask user)
-    (39 F.Mask user)
-    (44 Edge.Cuts user)
-    (45 Margin user)
-    (46 B.CrtYd user)
-    (47 F.CrtYd user)
-    (48 B.Fab user)
-    (49 F.Fab user)
+    (0 "F.Cu" signal "Top.Copper")
+    (1 "In1.Cu" power "Plane.1")
+    (2 "In2.Cu" power "Plane.2")
+    (31 "B.Cu" signal "Bottom.Copper")
+    (34 "B.Paste" user)
+    (35 "F.Paste" user)
+    (36 "B.SilkS" user "B.Silkscreen")
+    (37 "F.SilkS" user "F.Silkscreen")
+    (38 "B.Mask" user)
+    (39 "F.Mask" user)
+    (44 "Edge.Cuts" user)
+    (45 "Margin" user)
+    (46 "B.CrtYd" user "B.Courtyard")
+    (47 "F.CrtYd" user "F.Courtyard")
+    (48 "B.Fab" user)
+    (49 "F.Fab" user)
   )
   (setup
-    (last_trace_width 0.2)
-    (user_trace_width 0.25)
-    (user_trace_width 0.5)
-    (user_trace_width 0.75)
-    (user_trace_width 1)
-    (trace_clearance 0.25)
-    (zone_clearance 0.508)
-    (zone_45_only no)
-    (trace_min 0.15)
-    (via_size 0.5)
-    (via_drill 0.3)
-    (via_min_size 0.45)
-    (via_min_drill 0.3)
-    (user_via 0.5 0.3)
-    (user_via 0.9 0.5)
-    (uvia_size 0.3)
-    (uvia_drill 0.1)
-    (uvias_allowed no)
-    (uvia_min_size 0.2)
-    (uvia_min_drill 0.1)
-    (edge_width 0.05)
-    (segment_width 0.2)
-    (pcb_text_width 0.3)
-    (pcb_text_size 1.5 1.5)
-    (mod_edge_width 0.12)
-    (mod_text_size 1 1)
-    (mod_text_width 0.15)
-    (pad_size 1.524 1.524)
-    (pad_drill 0.762)
     (pad_to_mask_clearance 0.051)
     (solder_mask_min_width 0.25)
-    (aux_axis_origin 0 0)
-    (visible_elements 7FFFFFFF)
     (pcbplotparams
-      (layerselection 0x010fc_ffffffff)
+      (layerselection 0x00010fc_ffffffff)
+      (disableapertmacros false)
       (usegerberextensions false)
       (usegerberattributes false)
       (usegerberadvancedattributes false)
       (creategerberjobfile false)
+      (svguseinch false)
+      (svgprecision 6)
       (excludeedgelayer true)
-      (linewidth 0.100000)
       (plotframeref true)
       (viasonmask false)
@@
       (hpglpenspeed 20)
       (hpglpendiameter 15.000000)
+      (dxfpolygonmode true)
+      (dxfimperialunits true)
+      (dxfusepcbnewfont true)
       (psnegative false)
       (psa4output false)
@@
       (plotvalue true)
       (plotinvisibletext false)
-      (padsonsilk false)
+      (sketchpadsonfab false)
       (subtractmaskfromsilk false)
       (outputformat 4)
@@
       (drillshape 0)
       (scaleselection 1)
-      (outputdirectory ""))
+      (outputdirectory "")
+    )
   )
   (net 0 "")
-  (net_class Default "This is the default net class."
-    (clearance 0.25)
-    (trace_width 0.2)
-    (via_dia 0.5)
-    (via_drill 0.3)
-    (uvia_dia 0.3)
-    (uvia_drill 0.1)
-  )
 )
